File: LiDAR Interface Box.kicad_pcb (KiCad board)
At the start: 2 copper layers, 66 x 47 mm, 11 parts, among them J1 691214110002, J2 TSW-101-26-L-T, J3 PJ-102A, J4 691242710009, J5 SS-6488-NF, X1 01530007Z

Commit message: Updated text size on PCB
Other:
- board text added: "VLP-32C Power Supply V1.1"
- board text removed: "VLP-32 Power Supply V1.0"
Changed lines of the file:
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@@
   (gr_rect (start 81.28 54.61) (end 147.32 101.6) (layer "Edge.Cuts") (width 0.1) (fill none))
   (gr_text "GY" (at 110.381142 56.788857 270) (layer "F.SilkS")
-    (effects (font (size 0.5 0.5) (thickness 0.125)))
+    (effects (font (size 0.75 0.75) (thickness 0.125)))
   )
   (gr_text "BN" (at 125.512284 56.788857 270) (layer "F.SilkS")
-    (effects (font (size 0.5 0.5) (thickness 0.125)))
+    (effects (font (size 0.75 0.75) (thickness 0.125)))
   )
   (gr_text "WH" (at 130.556 56.788857 270) (layer "F.SilkS")
-    (effects (font (size 0.5 0.5) (thickness 0.125)))
+    (effects (font (size 0.75 0.75) (thickness 0.125)))
   )
   (gr_text "GN" (at 120.46857 56.788857 270) (layer "F.SilkS")
-    (effects (font (size 0.5 0.5) (thickness 0.125)))
+    (effects (font (size 0.75 0.75) (thickness 0.125)))
   )
   (gr_text "GND" (at 83.058 71.628) (layer "F.SilkS")
-    (effects (font (size 0.5 0.5) (thickness 0.125)))
+    (effects (font (size 0.5 0.75) (thickness 0.125)))
   )
   (gr_text "BU" (at 100.293714 56.788857 270) (layer "F.SilkS")
-    (effects (font (size 0.5 0.5) (thickness 0.125)))
+    (effects (font (size 0.75 0.75) (thickness 0.125)))
   )
   (gr_text "GND" (at 135.89 56.896 270) (layer "F.SilkS")
-    (effects (font (size 0.5 0.5) (thickness 0.125)))
+    (effects (font (size 0.75 0.75) (thickness 0.125)))
   )
   (gr_text "YE" (at 115.424856 56.788857 270) (layer "F.SilkS")
-    (effects (font (size 0.5 0.5) (thickness 0.125)))
+    (effects (font (size 0.75 0.75) (thickness 0.125)))
   )
   (gr_text "+12V" (at 83.058 75.438) (layer "F.SilkS")
-    (effects (font (size 0.5 0.5) (thickness 0.125)))
+    (effects (font (size 0.75 0.75) (thickness 0.125)))
   )
-  (gr_text "VLP-32 Power Supply\nV1.0" (at 107.95 96.266) (layer "F.SilkS")
+  (gr_text "VLP-32C Power Supply\nV1.1" (at 107.95 96.266) (layer "F.SilkS")
     (effects (font (size 1.5 1.5) (thickness 0.3)))
   )
   (gr_text "PK" (at 105.337428 56.788857 270) (layer "F.SilkS")
-    (effects (font (size 0.5 0.5) (thickness 0.125)))
+    (effects (font (size 0.75 0.75) (thickness 0.125)))
   )
   (gr_text "RD" (at 95.25 56.788857 270) (layer "F.SilkS")
-    (effects (font (size 0.5 0.5) (thickness 0.125)))
+    (effects (font (size 0.75 0.75) (thickness 0.125)))
   )
   (segment (start 112.835333 74.93) (end 124.205666 74.93) (width 3) (layer "F.Cu") (net 1))
